File: RFM69BreakoutBoard.sch (KiCad schematic (older format))
At the start: 4 parts

Commit message: updated schematic after talking with Chris
Parts:
- removed P?: CONN_1, ~, symbol CONN_1
- added C1: 1u, ~, symbol C
- added C2: 10u, ~, symbol C
- added C3, C4, C5, C6: .1u, ~, symbol C
- added C7: 10n, ~, symbol C
- added R4: 0, ~, symbol R
- added U1: MCP1703, ~, symbol MCP1703
- added U3: 74AHC1G, symbol 74AHC1G125
- added W1, W10, W2, W3, W4, W5, W6, W7, W8, W9: TEST, ~, symbol TEST
- U2: renamed from U?; value 74LVC245 -> 74LVC2; Distributor Part Number (none) -> 568-2274-1-ND; Distributor Part Number Link (none) -> http://www.digikey.com/product-detail/en/74LVC245ADB,118/56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; MFG Name (none) -> NXP Semiconductors; MFG Part Number (none) -> 74LVC245ADB,118
- U4: renamed from U?; Distributor Part Number (none) -> RFM69HW-433S2; Distributor Part Number Link (none) -> http://www.hoperfusa.com/details.jsp?pid=136; MFG Name (none) -> HopeRF; MFG Part Number (none) -> RFM69HW-433S2
- gave numbers to parts that had none: 1
Connections:
- net labels added: +5V, 5V, ANA, INT
- net labels removed: 3v3, IRQ
- wire segments 51 -> 79
Other:
- note added: "Arduino ->"
- moved on the sheet: P1, U2

Commit message: updated schema
Parts:
- removed R4: 0, ~, symbol R
- removed U4: RFM69HW, MODULE, symbol RFM69W
- added P?: CONN_1, ~, symbol CONN_1
- added U?: RFM69, MODULE, symbol RFM69
Connections:
- wire segments 79 -> 75
Other:
- note added: "hole for ant. wire"
Changed lines of the file:
@@
 LIBS:contrib
 LIBS:valves
-LIBS:RFM69W
-LIBS:mjAdditions
 LIBS:mcp1703
 LIBS:74AHC1G125
+LIBS:rfm69
 LIBS:RFM69BreakoutBoard-cache
 EELAYER 27 0
@@
 Sheet 1 1
 Title ""
-Date "24 feb 2014"
+Date "25 feb 2014"
 Rev ""
 Comp ""
@@
 Comment4 ""
 $EndDescr
-$Comp
-L RFM69W U4
-U 1 1 52FF74D2
-P 9000 4700
-F 0 "U4" H 9000 4600 50  0000 C CNN
-F 1 "RFM69HW" H 9000 4800 50  0000 C CNN
-F 2 "MODULE" H 9000 4700 50  0001 C CNN
-F 3 "DOCUMENTATION" H 9000 4700 50  0001 C CNN
-F 4 "HopeRF" H 9000 4700 60  0001 C CNN "MFG Name"
-F 5 "RFM69HW-433S2" H 9000 4700 60  0001 C CNN "MFG Part Number"
-F 6 "RFM69HW-433S2" H 9000 4700 60  0001 C CNN "Distributor Part Number"
-F 7 "http://www.hoperfusa.com/details.jsp?pid=136" H 9000 4700 60  0001 C CNN "Distributor Part Number Link"
-	1    9000 4700
-	-1   0    0    -1
-$EndComp
 $Comp
 L 74LVC245 U2
@@
 Text Label 1900 4700 0    60   ~ 0
 INT
-Text Label 8200 4950 0    60   ~ 0
+Text Label 7800 5050 0    60   ~ 0
 ANA
 Text Label 6650 4150 0    60   ~ 0
@@
 MISO
 $Comp
-L R R4
-U 1 1 53089115
-P 7900 4950
-F 0 "R4" V 7980 4950 40  0000 C CNN
-F 1 "0" V 7907 4951 31  0000 C CNN
-F 2 "~" V 7830 4950 30  0000 C CNN
-F 3 "~" H 7900 4950 30  0000 C CNN
-	1    7900 4950
-	0    -1   -1   0
-$EndComp
-$Comp
 L GND #PWR6
 U 1 1 530BB7C1
@@
 CS
 $Comp
-L GND #PWR9
-U 1 1 530BB991
-P 7500 5100
-F 0 "#PWR9" H 7500 5100 30  0001 C CNN
-F 1 "GND" H 7500 5030 30  0001 C CNN
-F 2 "" H 7500 5100 60  0000 C CNN
-F 3 "" H 7500 5100 60  0000 C CNN
-	1    7500 5100
-	1    0    0    -1
-$EndComp
-$Comp
 L +5V #PWR2
 U 1 1 530BBAA3
@@
 	1    0    0    -1
 $EndComp
-Wire Wire Line
-	6550 4050 6900 4050
-Wire Wire Line
-	1950 2300 2500 2300
-Wire Wire Line
-	1950 1900 1950 2600
-Wire Wire Line
-	3750 2300 9850 2300
-Wire Wire Line
-	3950 2300 3950 2600
-Wire Wire Line
-	4500 1950 4500 2300
-Connection ~ 3950 2300
-Connection ~ 4500 2300
-Wire Wire Line
-	3950 3150 3950 3000
-Connection ~ 3950 3150
-Wire Wire Line
-	3100 2800 3100 3150
-Connection ~ 3100 3150
-Wire Wire Line
-	1950 4100 1700 4100
-Wire Wire Line
-	1800 4200 1800 6050
-Wire Wire Line
-	1800 4200 1700 4200
-Wire Wire Line
-	1700 4700 2150 4700
-Wire Wire Line
-	2150 4700 2150 5950
-Wire Wire Line
-	9950 4450 9950 5950
-Wire Wire Line
-	9950 4450 9750 4450
-Wire Wire Line
-	7650 4150 7650 4750
-Wire Wire Line
-	7650 4750 8250 4750
-Wire Wire Line
-	7850 5050 8250 5050
-Wire Wire Line
-	7350 4650 8250 4650
-Wire Wire Line
-	7200 4450 8250 4450
-Wire Wire Line
-	9750 5050 9850 5050
-Wire Wire Line
-	6400 5600 7200 5600
-Wire Wire Line
-	7200 5600 7200 4450
-Wire Wire Line
-	7350 5500 7350 4650
-Wire Wire Line
-	4750 4400 4750 5400
-Wire Wire Line
-	4750 5400 5300 5400
-Wire Wire Line
-	5050 4500 5050 4150
-Wire Wire Line
-	5050 4150 5150 4150
-Wire Wire Line
-	8000 4250 8000 4550
-Wire Wire Line
-	8000 4550 8250 4550
-Wire Wire Line
-	5100 4600 5100 4250
-Wire Wire Line
-	5100 4250 5150 4250
-Wire Wire Line
-	8150 4350 8150 4450
-Connection ~ 8150 4450
-Connection ~ 1950 2300
-Wire Wire Line
-	4400 2600 4400 2300
-Connection ~ 4400 2300
-Wire Wire Line
-	6550 3950 6750 3950
-Wire Wire Line
-	1950 3000 1950 3150
-Wire Wire Line
-	8150 4950 8250 4950
-Wire Wire Line
-	8250 4850 8150 4850
-Wire Wire Line
-	8150 4850 8150 5050
-Connection ~ 8150 5050
-Wire Wire Line
-	7850 6050 7850 5050
-Wire Wire Line
-	5150 4850 4900 4850
-Wire Wire Line
-	4900 4850 4900 4950
-Wire Wire Line
-	7650 4950 7500 4950
-Wire Wire Line
-	7500 4950 7500 5100
-Wire Wire Line
-	4400 3000 4400 3600
-Wire Wire Line
-	1950 4100 1950 3800
-Wire Wire Line
-	1950 3150 4400 3150
-Connection ~ 4400 3150
-Wire Wire Line
-	4400 5600 4400 5450
-Wire Wire Line
-	5000 4050 5150 4050
-Wire Wire Line
-	5000 4300 5000 4050
-Wire Wire Line
-	1700 4300 3100 4300
-Wire Wire Line
-	3500 4300 5000 4300
-Wire Wire Line
-	4750 4400 3800 4400
-Wire Wire Line
-	3400 4400 1700 4400
-Wire Wire Line
-	3100 4500 1700 4500
-Wire Wire Line
-	3500 4500 5050 4500
-Wire Wire Line
-	3800 4600 5100 4600
-Wire Wire Line
-	3400 4600 1700 4600
-Wire Wire Line
-	1800 6050 3250 6050
-Wire Wire Line
-	3650 6050 7850 6050
-Wire Wire Line
-	2150 5950 3800 5950
-Wire Wire Line
-	9950 5950 4200 5950
-Wire Wire Line
-	6400 5400 6750 5400
-Wire Wire Line
-	6550 4150 7150 4150
-Wire Wire Line
-	7550 4150 7650 4150
-Wire Wire Line
-	6550 4250 6850 4250
-Wire Wire Line
-	7250 4250 8000 4250
 $Comp
 L TEST W7
@@
 	1    0    0    -1
 $EndComp
-Wire Wire Line
-	6400 5500 6750 5500
-Wire Wire Line
-	7150 5500 7350 5500
 $Comp
 L TEST W10
@@
 	1    0    0    -1
 $EndComp
-Wire Wire Line
-	6550 4350 7150 4350
-Wire Wire Line
-	7550 4350 8150 4350
 $Comp
 L C C5
@@
 	1    0    0    -1
 $EndComp
-Wire Wire Line
-	6750 2950 6750 2300
-Connection ~ 6750 2300
-Wire Wire Line
-	6750 3950 6750 3350
 $Comp
 L C C4
@@
 	0    -1   -1   0
 $EndComp
-Wire Wire Line
-	5050 5600 5300 5600
-Wire Wire Line
-	4400 5600 4650 5600
 $Comp
 L C C6
@@
 	1    0    0    -1
 $EndComp
-Wire Wire Line
-	9850 2300 9850 2950
 $Comp
 L C C7
@@
 	1    0    0    -1
 $EndComp
-Wire Wire Line
-	9850 3750 9850 3350
-Wire Wire Line
-	9850 3950 9850 4350
-Wire Wire Line
-	9850 4350 9750 4350
 Text Notes 550  4450 0    71   ~ 0
 Arduino ->
+$Comp
+L RFM69 U?
+U 1 1 530CA97F
+P 9000 4700
+F 0 "U?" H 9000 4600 50  0000 C CNN
+F 1 "RFM69" H 9000 4800 50  0000 C CNN
+F 2 "MODULE" H 9000 4300 50  0001 C CNN
+F 3 "DOCUMENTATION" H 9050 4200 50  0001 C CNN
+	1    9000 4700
+	-1   0    0    -1
+$EndComp
+$Comp
+L GND #PWR?
+U 1 1 530CAAF5
+P 1800 6350
+F 0 "#PWR?" H 1800 6350 30  0001 C CNN
+F 1 "GND" H 1800 6280 30  0001 C CNN
+F 2 "" H 1800 6350 60  0000 C CNN
+F 3 "" H 1800 6350 60  0000 C CNN
+	1    1800 6350
+	1    0    0    -1
+$EndComp
+Wire Wire Line
+	6550 4050 6900 4050
+Wire Wire Line
+	1950 2300 2500 2300
+Wire Wire Line
+	1950 1900 1950 2600
+Wire Wire Line
+	3750 2300 9850 2300
+Wire Wire Line
+	3950 2300 3950 2600
+Wire Wire Line
+	4500 1950 4500 2300
+Connection ~ 3950 2300
+Connection ~ 4500 2300
+Wire Wire Line
+	3950 3150 3950 3000
+Connection ~ 3950 3150
+Wire Wire Line
+	3100 2800 3100 3150
+Connection ~ 3100 3150
+Wire Wire Line
+	1950 4100 1700 4100
+Wire Wire Line
+	1800 4200 1800 6350
+Wire Wire Line
+	1800 4200 1700 4200
+Wire Wire Line
+	1700 4700 2150 4700
+Wire Wire Line
+	2150 4700 2150 5950
+Wire Wire Line
+	7650 4150 7650 4750
+Wire Wire Line
+	7650 4750 8250 4750
+Wire Wire Line
+	7350 4650 8250 4650
+Wire Wire Line
+	7200 4450 8250 4450
+Wire Wire Line
+	6400 5600 7200 5600
+Wire Wire Line
+	7200 5600 7200 4450
+Wire Wire Line
+	7350 5500 7350 4650
+Wire Wire Line
+	4750 4400 4750 5400
+Wire Wire Line
+	4750 5400 5300 5400
+Wire Wire Line
+	5050 4500 5050 4150
+Wire Wire Line
+	5050 4150 5150 4150
+Wire Wire Line
+	8000 4250 8000 4550
+Wire Wire Line
+	8000 4550 8250 4550
+Wire Wire Line
+	5100 4600 5100 4250
+Wire Wire Line
+	5100 4250 5150 4250
+Wire Wire Line
+	8150 4350 8150 4450
+Connection ~ 8150 4450
+Connection ~ 1950 2300
+Wire Wire Line
+	4400 2600 4400 2300
+Connection ~ 4400 2300
+Wire Wire Line
+	6550 3950 6750 3950
+Wire Wire Line
+	1950 3000 1950 3150
+Wire Wire Line
+	5150 4850 4900 4850
+Wire Wire Line
+	4900 4850 4900 4950
+Wire Wire Line
+	4400 3000 4400 3600
+Wire Wire Line
+	1950 4100 1950 3800
+Wire Wire Line
+	1950 3150 4400 3150
+Connection ~ 4400 3150
+Wire Wire Line
+	4400 5600 4400 5450
+Wire Wire Line
+	5000 4050 5150 4050
+Wire Wire Line
+	5000 4300 5000 4050
+Wire Wire Line
+	1700 4300 3100 4300
+Wire Wire Line
+	3500 4300 5000 4300
+Wire Wire Line
+	4750 4400 3800 4400
+Wire Wire Line
+	3400 4400 1700 4400
+Wire Wire Line
+	3100 4500 1700 4500
+Wire Wire Line
+	3500 4500 5050 4500
+Wire Wire Line
+	3800 4600 5100 4600
+Wire Wire Line
+	3400 4600 1700 4600
+Wire Wire Line
+	1800 6050 3250 6050
+Wire Wire Line
+	8000 6050 3650 6050
+Wire Wire Line
+	2150 5950 3800 5950
+Wire Wire Line
+	10550 5950 4200 5950
+Wire Wire Line
+	6400 5400 6750 5400
+Wire Wire Line
+	6550 4150 7150 4150
+Wire Wire Line
+	7550 4150 7650 4150
+Wire Wire Line
+	6550 4250 6850 4250
+Wire Wire Line
+	7250 4250 8000 4250
+Wire Wire Line
+	6400 5500 6750 5500
+Wire Wire Line
+	7150 5500 7350 5500
+Wire Wire Line
+	6550 4350 7150 4350
+Wire Wire Line
+	7550 4350 8150 4350
+Wire Wire Line
+	6750 2950 6750 2300
+Connection ~ 6750 2300
+Wire Wire Line
+	6750 3950 6750 3350
+Wire Wire Line
+	5050 5600 5300 5600
+Wire Wire Line
+	4400 5600 4650 5600
+Wire Wire Line
+	9850 2300 9850 2950
+Wire Wire Line
+	9850 3750 9850 3350
+Wire Wire Line
+	9850 3950 9850 5050
+Connection ~ 1800 6050
+Wire Wire Line
+	10550 4450 10550 5950
+$Comp
+L CONN_1 P?
+U 1 1 530CAD59
+P 7650 5050
+F 0 "P?" H 7730 5050 40  0000 L CNN
+F 1 "CONN_1" H 7650 5105 30  0001 C CNN
+F 2 "~" H 7650 5050 60  0000 C CNN
+F 3 "~" H 7650 5050 60  0000 C CNN
+	1    7650 5050
+	-1   0    0    1
+$EndComp
+Wire Wire Line
+	8000 4850 8000 6050
+Wire Wire Line
+	8000 4950 8250 4950
+Wire Wire Line
+	7800 5050 8250 5050
+Connection ~ 8000 5050
+Text Notes 7450 5200 0    60   ~ 0
+hole for ant. wire
+Wire Wire Line
+	8250 4850 8000 4850
+Connection ~ 8000 4950
+Wire Wire Line
+	9750 4450 10550 4450
+Wire Wire Line
+	9850 5050 9750 5050
 $EndSCHEMATC

Commit message: updated schema based on Sparkfun forum feedback
Parts:
- removed C4, C5, C6: .1u, ~, symbol C
- removed C7: 10n, ~, symbol C
- removed U3: 74AHC1G, symbol 74AHC1G125
- removed W1, W10, W2, W3, W4, W5, W6, W7, W8, W9: TEST, ~, symbol TEST
- added P10, P2, P3, P4, P5, P6, P7, P8, P9: TST, ~, symbol TST
- U2: value 74LVC2 -> 74LVC245
- U3: renamed from U?; value RFM69 -> RFM69HW
- gave numbers to parts that had none: 1
Connections:
- net labels added: CLK_3V3, CLK_5V, CS_3V3, CS_5V, MOSI_3V3, MOSI_5V
- net labels removed: ANA, CLK, CS, MOSI
- wire segments 75 -> 68

Commit message: added decoupling capacitors near RFM69, cleaned up GND
Parts:
- added C?: 10uF, ~, symbol C
- added C?: .1uF, ~, symbol C
- added D?: LED, ~, symbol LED
- added R?: 470, ~, symbol R
- added R?: 10K, ~, symbol R
Connections:
- wire segments 68 -> 79
Other:
- note added: "TBD: Antenna...."
- note removed: "hole for ant. wire"
- moved on the sheet: P4
Changed lines of the file:
@@
 Sheet 1 1
 Title ""
-Date "25 feb 2014"
+Date "26 feb 2014"
 Rev ""
 Comp ""
@@
 	1    0    0    -1
 $EndComp
-Wire Wire Line
-	1950 2300 2500 2300
-Wire Wire Line
-	1950 1900 1950 2600
-Wire Wire Line
-	3750 2300 9850 2300
-Wire Wire Line
-	3950 2300 3950 2600
-Wire Wire Line
-	4500 1950 4500 2300
-Connection ~ 3950 2300
-Connection ~ 4500 2300
-Wire Wire Line
-	3950 3150 3950 3000
-Connection ~ 3950 3150
-Wire Wire Line
-	3100 2800 3100 3150
-Connection ~ 3100 3150
-Wire Wire Line
-	1950 4100 1700 4100
-Wire Wire Line
-	1800 4200 1800 6350
-Wire Wire Line
-	1800 4200 1700 4200
-Wire Wire Line
-	1700 4700 2150 4700
-Wire Wire Line
-	2150 4700 2150 5950
-Wire Wire Line
-	7650 4150 7650 4750
-Wire Wire Line
-	7650 4750 8250 4750
-Wire Wire Line
-	7350 4650 8250 4650
-Wire Wire Line
-	7350 5400 7350 4650
-Wire Wire Line
-	4650 4400 4650 5400
-Wire Wire Line
-	4650 5400 7350 5400
-Wire Wire Line
-	4700 4500 4700 4150
-Wire Wire Line
-	4700 4150 5150 4150
-Wire Wire Line
-	8000 4250 8000 4550
-Wire Wire Line
-	8000 4550 8250 4550
-Wire Wire Line
-	4750 4600 4750 4250
-Wire Wire Line
-	4750 4250 5150 4250
-Wire Wire Line
-	8150 4350 8150 4450
-Connection ~ 1950 2300
-Wire Wire Line
-	4400 2600 4400 2300
-Connection ~ 4400 2300
-Wire Wire Line
-	6750 3950 6550 3950
-Wire Wire Line
-	1950 3000 1950 3150
-Wire Wire Line
-	4800 4850 5150 4850
-Wire Wire Line
-	4400 3000 4400 3600
-Wire Wire Line
-	1950 4100 1950 3800
-Wire Wire Line
-	1950 3150 4400 3150
-Connection ~ 4400 3150
-Wire Wire Line
-	4650 4050 5150 4050
-Wire Wire Line
-	4650 4300 4650 4050
-Wire Wire Line
-	1500 4300 4650 4300
-Wire Wire Line
-	1600 4400 4650 4400
-Wire Wire Line
-	1500 4500 4700 4500
-Wire Wire Line
-	1500 4600 4750 4600
-Wire Wire Line
-	8000 6050 1800 6050
-Wire Wire Line
-	2150 5950 10550 5950
-Wire Wire Line
-	6550 4150 7650 4150
-Wire Wire Line
-	6550 4250 8000 4250
-Wire Wire Line
-	6550 4350 8150 4350
-Wire Wire Line
-	6750 2300 6750 3950
-Connection ~ 6750 2300
-Wire Wire Line
-	9850 2300 9850 5050
-Connection ~ 1800 6050
-Wire Wire Line
-	10550 5950 10550 4450
 $Comp
 L CONN_1 P11
 U 1 1 530CAD59
-P 7650 4950
-F 0 "P11" H 7730 4950 40  0000 L CNN
-F 1 "CONN_1" H 7650 5005 30  0001 C CNN
-F 2 "~" H 7650 4950 60  0000 C CNN
-F 3 "~" H 7650 4950 60  0000 C CNN
-	1    7650 4950
+P 7750 5450
+F 0 "P11" H 7830 5450 40  0000 L CNN
+F 1 "CONN_1" H 7750 5505 30  0001 C CNN
+F 2 "~" H 7750 5450 60  0000 C CNN
+F 3 "~" H 7750 5450 60  0000 C CNN
+	1    7750 5450
 	-1   0    0    1
 $EndComp
-Wire Wire Line
-	8000 4850 8000 6050
-Text Notes 7400 4900 0    60   ~ 0
-hole for ant. wire
-Wire Wire Line
-	8000 4850 8250 4850
-Wire Wire Line
-	10550 4450 9750 4450
-Wire Wire Line
-	9850 5050 9750 5050
-Wire Wire Line
-	8150 4450 8250 4450
+Text Notes 7700 5600 0    60   ~ 0
+TBD: Antenna....
 $Comp
 L TST P6
@@
 	1    0    0    -1
 $EndComp
-Connection ~ 3700 4600
-Connection ~ 3400 4500
-Connection ~ 3150 4300
 $Comp
 L TST P5
@@
 	1    0    0    -1
 $EndComp
-Connection ~ 3550 4400
 $Comp
 L TST P7
@@
 L TST P4
 U 1 1 530D0696
-P 3400 6050
-F 0 "P4" H 3400 6350 40  0000 C CNN
-F 1 "TST" H 3400 6300 30  0000 C CNN
-F 2 "~" H 3400 6050 60  0000 C CNN
-F 3 "~" H 3400 6050 60  0000 C CNN
-	1    3400 6050
-	1    0    0    -1
-$EndComp
-Connection ~ 4000 5950
-Connection ~ 3400 6050
+P 3050 6050
+F 0 "P4" H 3050 6350 40  0000 C CNN
+F 1 "TST" H 3050 6300 30  0000 C CNN
+F 2 "~" H 3050 6050 60  0000 C CNN
+F 3 "~" H 3050 6050 60  0000 C CNN
+	1    3050 6050
+	1    0    0    -1
+$EndComp
 $Comp
 L TST P10
@@
 	1    0    0    -1
 $EndComp
+$Comp
+L R R?
+U 1 1 530DC938
+P 7300 4450
+F 0 "R?" V 7380 4450 40  0000 C CNN
+F 1 "470" V 7307 4451 40  0000 C CNN
+F 2 "~" V 7230 4450 30  0000 C CNN
+F 3 "~" H 7300 4450 30  0000 C CNN
+	1    7300 4450
+	0    -1   -1   0
+$EndComp
+$Comp
+L LED D?
+U 1 1 530DC956
+P 6800 4450
+F 0 "D?" H 6800 4550 50  0000 C CNN
+F 1 "LED" H 6800 4350 50  0000 C CNN
+F 2 "~" H 6800 4450 60  0000 C CNN
+F 3 "~" H 6800 4450 60  0000 C CNN
+	1    6800 4450
+	1    0    0    -1
+$EndComp
+$Comp
+L R R?
+U 1 1 530DCC1C
+P 2800 5050
+F 0 "R?" V 2880 5050 40  0000 C CNN
+F 1 "10K" V 2807 5051 40  0000 C CNN
+F 2 "~" V 2730 5050 30  0000 C CNN
+F 3 "~" H 2800 5050 30  0000 C CNN
+	1    2800 5050
+	1    0    0    -1
+$EndComp
+$Comp
+L +5V #PWR?
+U 1 1 530DCD57
+P 2800 5500
+F 0 "#PWR?" H 2800 5590 20  0001 C CNN
+F 1 "+5V" H 2800 5590 30  0000 C CNN
+F 2 "" H 2800 5500 60  0000 C CNN
+F 3 "" H 2800 5500 60  0000 C CNN
+	1    2800 5500
+	-1   0    0    1
+$EndComp
+$Comp
+L C C?
+U 1 1 530DFDC0
+P 10100 3650
+F 0 "C?" H 10100 3750 40  0000 L CNN
+F 1 "10uF" H 10106 3565 40  0000 L CNN
+F 2 "~" H 10138 3500 30  0000 C CNN
+F 3 "~" H 10100 3650 60  0000 C CNN
+	1    10100 3650
+	1    0    0    -1
+$EndComp
+$Comp
+L GND #PWR?
+U 1 1 530DFEA1
+P 10100 4050
+F 0 "#PWR?" H 10100 4050 30  0001 C CNN
+F 1 "GND" H 10100 3980 30  0001 C CNN
+F 2 "" H 10100 4050 60  0000 C CNN
+F 3 "" H 10100 4050 60  0000 C CNN
+	1    10100 4050
+	1    0    0    -1
+$EndComp
+$Comp
+L C C?
+U 1 1 530DFF22
+P 10550 3650
+F 0 "C?" H 10550 3750 40  0000 L CNN
+F 1 ".1uF" H 10556 3565 40  0000 L CNN
+F 2 "~" H 10588 3500 30  0000 C CNN
+F 3 "~" H 10550 3650 60  0000 C CNN
+	1    10550 3650
+	1    0    0    -1
+$EndComp
+Wire Wire Line
+	1950 2300 2500 2300
+Wire Wire Line
+	1950 1900 1950 2600
+Wire Wire Line
+	3750 2300 9850 2300
+Wire Wire Line
+	3950 2300 3950 2600
+Wire Wire Line
+	4500 1950 4500 2300
+Connection ~ 3950 2300
+Connection ~ 4500 2300
+Wire Wire Line
+	3950 3150 3950 3000
+Connection ~ 3950 3150
+Wire Wire Line
+	3100 2800 3100 3150
+Connection ~ 3100 3150
+Wire Wire Line
+	1950 4100 1700 4100
+Wire Wire Line
+	1800 4200 1800 6350
+Wire Wire Line
+	1800 4200 1700 4200
+Wire Wire Line
+	1700 4700 2150 4700
+Wire Wire Line
+	2150 4700 2150 5950
+Wire Wire Line
+	7650 4150 7650 4750
+Wire Wire Line
+	7650 4750 8250 4750
+Wire Wire Line
+	7350 4650 8250 4650
+Wire Wire Line
+	7350 5400 7350 4650
+Wire Wire Line
+	4650 4400 4650 5400
+Wire Wire Line
+	4650 5400 7350 5400
+Wire Wire Line
+	4700 4500 4700 4150
+Wire Wire Line
+	4700 4150 5150 4150
+Wire Wire Line
+	8000 4250 8000 4550
+Wire Wire Line
+	8000 4550 8250 4550
+Wire Wire Line
+	4750 4600 4750 4250
+Wire Wire Line
+	4750 4250 5150 4250
+Wire Wire Line
+	8150 4350 8150 4450
+Connection ~ 1950 2300
+Wire Wire Line
+	4400 2600 4400 2300
+Connection ~ 4400 2300
+Wire Wire Line
+	6750 3950 6550 3950
+Wire Wire Line
+	1950 3000 1950 3150
+Wire Wire Line
+	4800 4850 5150 4850
+Wire Wire Line
+	4400 3000 4400 3600
+Wire Wire Line
+	1950 4100 1950 3800
+Wire Wire Line
+	1950 3150 4400 3150
+Connection ~ 4400 3150
+Wire Wire Line
+	4650 4050 5150 4050
+Wire Wire Line
+	4650 4300 4650 4050
+Wire Wire Line
+	1500 4300 4650 4300
+Wire Wire Line
+	1600 4400 4650 4400
+Wire Wire Line
+	1500 4500 4700 4500
+Wire Wire Line
+	1500 4600 4750 4600
+Wire Wire Line
+	7400 6050 1800 6050
+Wire Wire Line
+	2150 5950 10550 5950
+Wire Wire Line
+	6550 4150 7650 4150
+Wire Wire Line
+	6550 4250 8000 4250
+Wire Wire Line
+	6550 4350 8150 4350
+Wire Wire Line
+	6750 2300 6750 3950
+Connection ~ 6750 2300
+Wire Wire Line
+	9850 2300 9850 5050
+Wire Wire Line
+	10550 5950 10550 4450
+Wire Wire Line
+	7400 4850 7400 6050
+Wire Wire Line
+	7400 4850 8250 4850
+Wire Wire Line
+	10550 4450 9750 4450
+Wire Wire Line
+	9850 5050 9750 5050
+Wire Wire Line
+	8150 4450 8250 4450
+Connection ~ 3700 4600
+Connection ~ 3400 4500
+Connection ~ 3150 4300
+Connection ~ 3550 4400
+Connection ~ 4000 5950
 Connection ~ 7300 4350
 Connection ~ 7200 4250
 Connection ~ 7350 4150
 Wire Wire Line
-	7800 4950 8250 4950
-Connection ~ 8000 4950
-Wire Wire Line
-	8250 5050 8000 5050
-Connection ~ 8000 5050
+	7400 5050 8250 5050
 Wire Wire Line
 	5050 4750 5150 4750
@@
 	4950 4650 5150 4650
 Wire Wire Line
-	4800 4350 4800 4950
-Wire Wire Line
 	4900 4550 5150 4550
 Wire Wire Line
-	4800 4350 5150 4350
+	4500 4350 5150 4350
 Wire Wire Line
 	5150 3950 5150 2300
@@
 	5050 4750 5050 4850
 Connection ~ 5050 4850
-Connection ~ 4800 4850
 Wire Wire Line
 	6550 4050 6800 4050
@@
 Wire Wire Line
 	6950 3850 6950 3950
+Wire Wire Line
+	4800 4850 4800 4950
+Wire Wire Line
+	4500 4350 4500 4300
+Connection ~ 4500 4300
+Wire Wire Line
+	6550 4450 6600 4450
+Wire Wire Line
+	7000 4450 7050 4450
+Wire Wire Line
+	7550 4450 7550 4350
+Connection ~ 7550 4350
+Wire Wire Line
+	2800 4800 2800 4600
+Connection ~ 2800 4600
+Wire Wire Line
+	2800 5300 2800 5500
+Connection ~ 1800 6050
+Connection ~ 3050 6050
+Connection ~ 7400 5050
+Wire Wire Line
+	10100 3850 10100 4050
+Wire Wire Line
+	10550 3850 10550 3950
+Wire Wire Line
+	10550 3950 10100 3950
+Connection ~ 10100 3950
+Wire Wire Line
+	10100 3450 10100 3300
+Wire Wire Line
+	9850 3300 10550 3300
+Connection ~ 9850 3300
+Wire Wire Line
+	10550 3300 10550 3450
+Connection ~ 10100 3300
 $EndSCHEMATC

Commit message: edited antenna pin in schematic
Parts:
- removed P11: CONN_1, ~, symbol CONN_1
- added P?: ANA hole, ~, symbol TST
Connections:
- wire segments 79 -> 89
Other:
- note removed: "TBD: Antenna...."
Changed lines of the file:
@@
 $EndComp
-$Comp
-L CONN_1 P11
-U 1 1 530CAD59
-P 7750 5450
-F 0 "P11" H 7830 5450 40  0000 L CNN
-F 1 "CONN_1" H 7750 5505 30  0001 C CNN
-F 2 "~" H 7750 5450 60  0000 C CNN
-F 3 "~" H 7750 5450 60  0000 C CNN
-	1    7750 5450
-	-1   0    0    1
-$EndComp
-Text Notes 7700 5600 0    60   ~ 0
-TBD: Antenna....
 $Comp
 L TST P6
@@
 	10550 3300 10550 3450
 Connection ~ 10100 3300
+$Comp
+L TST P?
+U 1 1 530E5A0D
+P 7750 6650
+F 0 "P?" H 7750 6950 40  0000 C CNN
+F 1 "ANA hole" H 7750 6900 30  0000 C CNN
+F 2 "~" H 7750 6650 60  0000 C CNN
+F 3 "~" H 7750 6650 60  0000 C CNN
+	1    7750 6650
+	-1   0    0    1
+$EndComp
+Wire Wire Line
+	8250 4950 7750 4950
+Wire Wire Line
+	7750 4950 7750 6650
+$Comp
+L GND #PWR?
+U 1 1 530E5AC0
+P 8100 6450
+F 0 "#PWR?" H 8100 6450 30  0001 C CNN
+F 1 "GND" H 8100 6380 30  0001 C CNN
+F 2 "" H 8100 6450 60  0000 C CNN
+F 3 "" H 8100 6450 60  0000 C CNN
+	1    8100 6450
+	1    0    0    -1
+$EndComp
+Wire Wire Line
+	7750 6400 8100 6400
+Wire Wire Line
+	8100 6400 8100 6450
+Connection ~ 7750 6400
+$Comp
+L GND #PWR?
+U 1 1 530E5B36
+P 8100 6300
+F 0 "#PWR?" H 8100 6300 30  0001 C CNN
+F 1 "GND" H 8100 6230 30  0001 C CNN
+F 2 "" H 8100 6300 60  0000 C CNN
+F 3 "" H 8100 6300 60  0000 C CNN
+	1    8100 6300
+	1    0    0    -1
+$EndComp
+Wire Wire Line
+	7750 6250 8100 6250
+Connection ~ 7750 6250
+$Comp
+L GND #PWR?
+U 1 1 530E5BAF
+P 8100 6150
+F 0 "#PWR?" H 8100 6150 30  0001 C CNN
+F 1 "GND" H 8100 6080 30  0001 C CNN
+F 2 "" H 8100 6150 60  0000 C CNN
+F 3 "" H 8100 6150 60  0000 C CNN
+	1    8100 6150
+	1    0    0    -1
+$EndComp
+Wire Wire Line
+	7750 6100 8100 6100
+Connection ~ 7750 6100
+Wire Wire Line
+	8100 6100 8100 6150
+Wire Wire Line
+	8100 6250 8100 6300
+$Comp
+L GND #PWR?
+U 1 1 530E5DE4
+P 8100 6650
+F 0 "#PWR?" H 8100 6650 30  0001 C CNN
+F 1 "GND" H 8100 6580 30  0001 C CNN
+F 2 "" H 8100 6650 60  0000 C CNN
+F 3 "" H 8100 6650 60  0000 C CNN
+	1    8100 6650
+	1    0    0    -1
+$EndComp
+Wire Wire Line
+	7750 6550 8100 6550
+Wire Wire Line
+	8100 6550 8100 6650
+Connection ~ 7750 6550
 $EndSCHEMATC
