File: _autosave-RFM69BreakoutBoard.kicad_pcb (KiCad board)
At the start: 2 copper layers, 26.2 x 25.8 mm, 21 parts, among them P1 BB Holes, P10 TST, P11 TST, P12 TST, P2 TST, P3 TST, P4 TST, P5 TST, P6 TST, P7 TST, P8 TST, P9 TST, U1 MCP1703, U2 74HCT123, U3 RFM69HW

Commit message: updated BOM
Parts:
- moved P12 9.28 mm to (105.4, 150.7)
- moved C5 9.17 mm to (80.4, 148.3), turned to 90 degrees
- moved C1 9.05 mm to (98.7, 146.6), turned to 90 degrees
- moved C2 8.75 mm to (86.4, 148.6), turned to 90 degrees
- moved U1 8.56 mm to (89.3, 145.0), turned to 270 degrees
- moved C3 5.77 mm to (84.2, 148.5), turned to 90 degrees
- moved P11 4.71 mm to (105.5, 154.9)
- moved P10 4.31 mm to (105.7, 157.1)
- moved P9 4.26 mm to (105.7, 159.0)
- moved R1 3.99 mm to (95.8, 146.9)
- moved U2 3.75 mm to (94.0, 153.9), turned to 0 degrees
- moved P8 3.66 mm to (105.7, 161.2)
- moved C4 3.51 mm to (82.3, 148.5)
- moved U3 3.14 mm to (94.1, 147.7)
- moved P4 1.49 mm to (96.9, 160.0)
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Routing:
- net GND: track 73.3 -> 0.00 mm, vias 2 -> 0
- net +3.3V: track 36.0 -> 0.00 mm, vias 2 -> 0
- net +5V: track 28.6 -> 0.00 mm
- net /CS_5V: track 21.4 -> 0.00 mm
- net /MOSI_5V: track 16.9 -> 0.00 mm
- net /CLK_3V3: track 15.2 -> 0.00 mm, vias 1 -> 0
- net /MISO: track 15.1 -> 0.00 mm
- net /CS_3V3: track 10.8 -> 0.00 mm, vias 1 -> 0
- net /MISO_3V3: track 10.1 -> 0.00 mm, vias 1 -> 0
- net /INT: track 9.92 -> 0.00 mm
- net /ANA: track 7.32 -> 0.00 mm
- net /MOSI_3V3: track 3.42 -> 0.00 mm
