File: $RFM69BreakoutBoard.sch (KiCad schematic (older format))
At the start: 21 parts, among them P1 BB Holes, P10 TST, P11 TST, P12 TST, P2 TST, P3 TST, P4 TST, P5 TST, P6 TST, P7 TST, P8 TST, P9 TST, U1 MCP1703, U2 74HCT123, U3 RFM69HW

Commit message: first pass of trace
Connections:
- net CS_5V: now also P7.1
Changed lines of the file:
@@
 	3200 4000 3200 4500
-Wire Wire Line
-	3400 4000 3400 4600
 Wire Wire Line
 	2250 6300 2250 6050
@@
 	4400 4400 4400 5200
 Wire Wire Line
-	5900 5200 4400 5200
+	4400 5200 5900 5200
 Wire Wire Line
-	5900 4900 5900 5200
+	5900 5200 5900 4900
 Connection ~ 3000 4400
+Wire Wire Line
+	3400 4000 3400 4600
+Connection ~ 3400 4600
 $EndSCHEMATC
